File: pcb_canfd/canfd_transducer/canfd_transducer.kicad_pcb (KiCad board)
At the start: 2 copper layers, 7 parts, among them J1 Conn_01x13_Female, J2 Conn_01x03_Female, U1 MCP2517FD-xSL

Commit message: finished first version of board, needs revision
Parts:
- added H1: MountingHole, MountingHole:MountingHole_3.2mm_M3_DIN965_Pad_TopOnly, F.Cu at (149.9, 83.8)
- added H2: MountingHole, MountingHole:MountingHole_3.2mm_M3_DIN965_Pad_TopOnly, F.Cu at (149.9, 63.5)
- added H3: MountingHole, MountingHole:MountingHole_3.2mm_M3_DIN965_Pad_TopOnly, F.Cu at (104.1, 63.5)
- added H4: MountingHole, MountingHole:MountingHole_3.2mm_M3_DIN965_Pad_TopOnly, F.Cu at (104.1, 83.8)
- J1: footprint Connector_PinHeader_2.54mm:PinHeader_1x13_P2.54mm_Vertical -> Connector_PinSocket_2.54mm:PinSocket_1x13_P2.54mm_Vertical; moved to B.Cu
- J2: moved to B.Cu
- moved C3 49.6 mm to (127.2, 68.9), turned to -90 degrees
- moved J1 37.1 mm to (139.7, 82.2), turned to 90 degrees
- moved J2 30.1 mm to (141.1, 75.3), turned to 90 degrees
- moved C1 16.6 mm to (135.4, 79.2), turned to 180 degrees
- moved C2 14.8 mm to (139.7, 66.9), turned to -90 degrees
- moved U2 6.35 mm to (132.1, 68.6), turned to -90 degrees
- moved U1 3.59 mm to (121.9, 73.7)
- renumbered 11 to U2
Connections:
- J1 pad 11: /~{INT1} -> /OSC2
- J1 pad 12: /~{INT0} -> /~{INT}
- J1 pad 13: /~{INT} -> /CLKO
- J1 pad 2: +3.3V -> GND
- J1 pad 3: GND -> +3.3V
- J1 pad 4: /SDI -> /nCS
- J1 pad 6: /nCS -> /SDI
- J1 pad 8: /CLKO -> /~{INT0}
- J1 pad 9: /OSC2 -> /~{INT1}
- J2 pad 1: unconnected-(J2-Pad1) -> /CANH
- J2 pad 2: /CANH -> /CANL
- J2 pad 3: /CANL -> GND
Routing:
- net GND: track 0.00 -> 89.9 mm
- net +5V: track 0.00 -> 31.9 mm
- net /CAN_TX: track 0.00 -> 19.5 mm
- net +3.3V: track 0.00 -> 19.3 mm
- net /CLKO: track 0.00 -> 16.3 mm
- net /nCS: track 0.00 -> 15.6 mm
- net /CAN_RX: track 0.00 -> 14.1 mm
- net /~{INT}: track 0.00 -> 13.3 mm
- net /SDO: track 0.00 -> 12.7 mm
- net /CANH: track 0.00 -> 12.0 mm
- net /SDI: track 0.00 -> 11.3 mm
- net /OSC2: track 0.00 -> 10.4 mm
- net /SCK: track 0.00 -> 9.97 mm
- net /CANL: track 0.00 -> 9.71 mm
- net /~{INT0}: track 0.00 -> 8.82 mm
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- added copper zone on F.Cu, net GND
Other:
- board outline added: 55.9 x 30.5 mm
- board text added: "3.3V"
- board text added: "5V"
- board text added: "CLKO"
- board text added: "G"
- board text added: "GND"
- board text added: "H"
- board text added: "L"
- board text added: "OSC1"
- board text added: "OSC2"
- board text added: "SCK"
- board text added: "SDI"
- board text added: "SDO"
- board text added: "nCS"
- board text added: "~{INT0}"
- board text added: "~{INT1}"
- board text added: "~{INT}"

Commit message: added resistor for can bus
Parts:
- added R1: 120ohm, Resistor_SMD:R_0805_2012Metric, F.Cu at (136.6, 73.4)
- moved J2 3.24 mm to (140.6, 72.1), turned to -90 degrees
Connections:
- U2 pad 6: /CANH -> /CANL
- U2 pad 7: /CANL -> /CANH
Routing:
- net GND: track 89.9 -> 84.0 mm
- net /CANH: track 12.0 -> 9.79 mm
- net /CANL: track 9.71 -> 11.2 mm
